Commit message: fully defined robot

File: src/scara_params/urdf/scara.urdf (robot description, URDF)
Before this commit: robot arm, 2 links, 1 joints
Links:
- added link link_2, mass 1.0; collision box size=1.0 0.08 0.08; collision sphere radius=0.08
- added link tool_link, mass 0.5; collision box size=0.1 0.1 0.1; visual box size=0.1 0.1 0.1
- link base: geometry collision sphere radius=0.08; visual box size=0.3 0.3 0.1
Joints:
- added joint joint_2: type revolute, parent link_1, child link_2, origin xyz=1.0 0 1.0 rpy=0 0 0, axis 0 0 1, limit lower=-3.14 upper=3.14 effort=20 velocity=1
- added joint joint_3: type prismatic, parent link_2, child tool_link, origin xyz=1.0 0 0 rpy=0 0 0, axis 0 0 -1, limit lower=0.0 upper=0.5 effort=20 velocity=0.25
- joint joint_1: origin xyz=0 0 0.35 rpy=0 0 0 -> xyz=0 0 0 rpy=0 0 0
